File: PCB/Orthrus-TX.kicad_pcb (KiCad board)
At the start: 8 copper layers, 49 x 49 mm, 158 parts, among them J1 HRO-TYPE-C-31-M-13x, U1 AO3407A, U2 SRV05-4, U3 SRV05-4, U4 SRV05-4, U5 SRV05-4, U6 SRV05-4, U7 SRV05-4, U8 SRV05-4

Commit message: pcb update
Parts:
- U2, U3, U4, U5, U6, U7, U8: footprint Package_TO_SOT_SMD:SOT-23-6 -> Custom-Library:SOT-23-6
- moved U2 0.34 mm to (132.3, 55.9), turned to -90 degrees
- moved C55 0.22 mm to (161.3, 70.4)
- moved U5 0.21 mm to (164.8, 71.7)
- moved L2 0.19 mm to (130.9, 61.6)
Connections:
- net /USB_N_OUT renamed /USB_D_N
- net /USB_P_OUT renamed /USB_D_P
- ELRS_1 pad 4: GND -> /PD9
- ELRS_1 pad 5: /PD9 -> GND
- ELRS_1 pad 6: GND -> /PD10
- ELRS_1 pad 7: /PD10 -> /PD11
- ELRS_1 pad 8: /PD11 -> GND
- ELRS_2 pad 4: GND -> /PE7
- ELRS_2 pad 5: /PE7 -> GND
- ELRS_2 pad 6: GND -> /PB5
- ELRS_2 pad 7: /PB5 -> /PB8
- ELRS_2 pad 8: /PB8 -> GND
- U5 pad 1: /PD8 -> /PD9
- U5 pad 3: /PD9 -> /PD8
- U5 pad 4: /PD10 -> /PD11
- U5 pad 6: /PD11 -> /PD10
- U6 pad 4: /PB5 -> /PB8
- U6 pad 6: /PB8 -> /PB5
Routing:
- net /USB_P: track 6.94 -> 13.6 mm, vias 2 -> 3
- net /LD1_3.3v: track 288.7 -> 283.7 mm, vias 34 -> 35
- net /PE8: track 27.9 -> 23.6 mm
- net /USB_N: track 9.83 -> 13.6 mm, vias 2 -> 3
- net /PB5: track 47.0 -> 43.3 mm, vias 3 -> 2
- net /PD11: track 18.9 -> 15.4 mm
- net Net-(D1-A): track 24.3 -> 27.2 mm
- net /PB8: track 45.5 -> 43.2 mm, vias 3 -> 2
- net /PD8: track 21.1 -> 19.2 mm
- net /PD9: track 16.5 -> 18.0 mm
- net /PE7: track 26.0 -> 25.1 mm
- net /PD10: track 15.8 -> 15.0 mm
- net GND: vias 83 -> 86

Commit message: Update Orthrus-TX.kicad_pcb
Routing:
- net /PC7: track 22.5 -> 20.6 mm
- net /PC6: track 18.7 -> 17.4 mm
- net /PC9: track 24.8 -> 24.3 mm
- net GND: vias 86 -> 95

Commit message: pcb update
Parts:
- U2: moved to B.Cu
- moved L2 6.80 mm to (131.8, 54.9), turned to 90 degrees
- moved U2 2.60 mm to (132.7, 58.5), turned to 0 degrees
- moved C6 0.91 mm to (132.8, 59.6)
- moved C23 0.89 mm to (132.5, 61.8)
- moved C22 0.42 mm to (135.0, 58.0)
- moved C4 0.30 mm to (133.9, 51.0)
- moved C5 0.30 mm to (133.9, 52.5)
- moved C54 0.30 mm to (133.7, 49.5)
Connections:
- U2 pad 1: /USB_P -> /USB_N
- U2 pad 3: /USB_N -> /USB_P
Routing:
- net Net-(D1-A): track 27.2 -> 32.0 mm, vias 3 -> 4
- net /USB_N: track 13.6 -> 9.25 mm, vias 3 -> 2
- net /USB_P: track 13.6 -> 9.38 mm, vias 3 -> 2
- net /USB_D_P: track 33.5 -> 29.5 mm
- net /USB_D_N: track 32.6 -> 30.7 mm
- net /LD1_3.3v: track 283.7 -> 282.2 mm
- net Net-(J1-CC2): track 8.62 -> 9.57 mm
- net /VCAP: track 66.3 -> 65.7 mm
- net /NRST: track 44.9 -> 44.5 mm, vias 4 -> 3
- net /PE9: vias 2 -> 4
- net GND: vias 95 -> 94

Commit message: Update Orthrus-TX.kicad_pcb
Routing:
- net /PG11: track 26.2 -> 29.8 mm
- net /PG13: track 19.2 -> 21.9 mm
- net /PG12: track 26.8 -> 26.1 mm, vias 2 -> 3

Commit message: sd card routing update
Parts:
- moved C53 25.3 mm to (133.6, 26.8)
- moved U4 25.3 mm to (134.0, 24.2)
- moved R47 16.1 mm to (162.3, 52.8), turned to -90 degrees
- moved U3 14.9 mm to (151.8, 40.3), turned to -90 degrees
- moved C51 12.2 mm to (160.9, 36.2), turned to 180 degrees
- moved R50 9.70 mm to (167.5, 37.4), turned to 90 degrees
- moved C50 9.10 mm to (160.9, 37.7), turned to 180 degrees
- moved R41 5.70 mm to (135.3, 67.7)
- moved R51 5.25 mm to (155.1, 52.4), turned to 0 degrees
- moved C52 3.95 mm to (151.9, 43.9), turned to 90 degrees
- moved R42 2.65 mm to (135.3, 66.1)
- moved R48 2.40 mm to (164.9, 36.7)
- moved R49 2.19 mm to (163.2, 37.0)
- moved R46 1.91 mm to (163.8, 52.8)
- moved R45 1.74 mm to (165.4, 53.1)
Routing:
- net /PB14: track 51.0 -> 6.92 mm, vias 6 -> 1
- net /PB15: track 44.2 -> 6.76 mm, vias 7 -> 1
- net /LD4_3.3v: track 86.7 -> 58.1 mm, vias 6 -> 2
- net /PD7: track 36.3 -> 9.42 mm, vias 4 -> 1
- net /PG11: track 29.8 -> 6.89 mm, vias 3 -> 1
- net /PG12: track 26.1 -> 7.52 mm, vias 3 -> 1
- net /PG13: track 21.9 -> 3.71 mm
- net /SD_CLK: track 22.1 -> 6.44 mm, vias 3 -> 0
- net /PD6: track 12.6 -> 1.22 mm, vias 2 -> 1
- net Net-(J1-CC1): track 10.9 -> 13.3 mm
- net Net-(J1-CC2): track 9.57 -> 10.9 mm
