File: PCB/Orthrus-TX.kicad_sch (KiCad schematic)
At the start: 157 parts, among them J1 HRO-TYPE-C-31-M-13x, U1 AO3407A, U2 SRV05-4, U3 SRV05-4, U4 SRV05-4, U5 SRV05-4, U6 SRV05-4, U7 SRV05-4, U8 SRV05-4

Commit message: pcb update
Parts:
- C19, C45: value 100nF -> 10nF; LCSC C24452 -> C3836718
Connections:
- net LD2_3.3v: no longer R54.1
- net VDDA: now also R54.1
Other:
- moved on the sheet: C19, C20, C45, C46, L3, R54

Commit message: pcb update
Parts:
- added R58, R59, R60, R61, R62: 33Ω, Resistor_SMD:R_0603_1608Metric, symbol Device:R_US
Connections:
- net GND: now also U2.4 (IO3), U2.6 (IO4), U4.4 (IO3), U8.4 (IO3), U8.6 (IO4)
- net PB14: now also R62.1; no longer SD_CARD_1.7 (DAT0)
- net PB15: now also R61.1; no longer SD_CARD_1.8 (DAT1)
- net PD7: now also R60.2; no longer SD_CARD_1.3 (CMD)
- net PG11: now also R58.2; no longer SD_CARD_1.1 (DAT2)
- net PG12: now also R59.2; no longer SD_CARD_1.2 (CD/DAT3)
- new net: R59.1, SD_CARD_1.2 (CD/DAT3)
- new net: R61.2, SD_CARD_1.8 (DAT1)
- new net: R58.1, SD_CARD_1.1 (DAT2)
- new net: R60.1, SD_CARD_1.3 (CMD)
- new net: R62.2, SD_CARD_1.7 (DAT0)

Commit message: pcb update
Parts:
- removed D1: D_Schottky, Diode_SMD:D_SOD-123, symbol Device:D_Schottky
- removed POWER_1: 532610371, Custom-Library:CONN_532610001-SD_03_MOL, symbol CONN_532610001-SD_03_MOL:532610371
- added POWER_1: 532610571, CONN_532610001-SD_05_MOL, symbol CONN_532610001-SD_05_MOL:532610571
Connections:
- net BATT_IN: now also POWER_1.2
- net GND: now also POWER_1.1, POWER_1.4
- net LD1_3.3v: now also C54.2, U2.5 (VP)
- net RAW: now also POWER_1.3
- net BATT_CHARGE: now reaches J1.A4 (VBUS), J1.A9 (VBUS), J1.B4 (VBUS), J1.B9 (VBUS)
- net BATT_CHARGE: now also POWER_1.5; no longer C54.2, U2.5 (VP)
Other:
- moved on the sheet: R57, U1
